File: circuit/main.kicad_pcb (KiCad board)
At the start: 2 copper layers, 76.2 x 38.1 mm, 28 parts, among them IC1 PIC16F1778-I_SP, J1 Conn_01x06_Pin, J2 Conn_01x06_Pin, M1 Motor_DC, M2 Motor_DC, Q1 MP4212_Q_, Q2 MP4212_Q_, SW1 SW_SPDT

Commit message: circuit rc2
Parts:
- moved BT1 1.27 mm to (85.1, 35.6)
- moved C3 1.27 mm to (74.9, 27.2)
- moved C4 1.27 mm to (80.0, 25.4)
- moved R2 1.27 mm to (66.0, 34.3)
- moved REF** 1.27 mm to (85.1, 45.7)
- moved REF** 1.27 mm to (85.1, 17.8)
- moved SW1 1.27 mm to (85.1, 27.9)
- moved D1 1.27 mm to (52.1, 39.4)
- moved J2 1.27 mm to (44.5, 39.4)
- moved Q1 1.27 mm to (52.1, 21.6)
- moved Q2 1.27 mm to (47.0, 21.6)
- moved R4 1.27 mm to (52.1, 41.9)
- moved REF** 1.27 mm to (49.5, 16.5)
- moved R1 1.27 mm to (16.5, 31.8)
- moved C2 1.27 mm to (19.1, 19.1)
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Other:
- board size 76.2 x 38.1 mm -> 77.5 x 38.1 mm
